File: Super Nano/sg_model2-3_s-video_supernano.kicad_pcb (KiCad board)
At the start: 2 copper layers, 9.4 x 7.5 mm, 10 parts, among them J1 Y-I, J2 C-I, J3 Y-O, J4 C-O, J5 GND, J6 GND

Commit message: super nano - minor update
Routing:
- net GND: track 7.34 -> 0.01 mm
Other:
- board text added: "YCGND"
Changed lines of the file:
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@@
     (fp_line (start 1 0.625) (end -1 0.625)
       (stroke (width 0.1) (type solid)) (layer "F.Fab"))
-    (pad "1" smd roundrect (at -0.9125 0) (size 1.025 1.4) (layers "F.Cu" "F.Paste" "F.Mask") (roundrect_rratio 0.243902)
+    (pad "1" smd roundrect (at -0.9125 0) (size 1.025 1.4) (layers "F.Cu" "F.Paste" "F.Mask") (roundrect_rratio 0.243902439)
       (net 6 "Net-(J2-Pin_1)") (pintype "passive"))
-    (pad "2" smd roundrect (at 0.9125 0) (size 1.025 1.4) (layers "F.Cu" "F.Paste" "F.Mask") (roundrect_rratio 0.243902)
+    (pad "2" smd roundrect (at 0.9125 0) (size 1.025 1.4) (layers "F.Cu" "F.Paste" "F.Mask") (roundrect_rratio 0.243902439)
       (net 3 "Net-(C2-Pad1)") (pintype "passive"))
     (model "${KICAD6_3DMODEL_DIR}/Resistor_SMD.3dshapes/R_0805_2012Metric.wrl"
@@
     (fp_line (start 1.75 1.4) (end 1.75 -1.4)
       (stroke (width 0.1) (type solid)) (layer "F.Fab"))
-    (pad "1" smd roundrect (at -1.5375 0) (size 1.325 2.35) (layers "F.Cu" "F.Paste" "F.Mask") (roundrect_rratio 0.188679)
+    (pad "1" smd roundrect (at -1.5375 0) (size 1.325 2.35) (layers "F.Cu" "F.Paste" "F.Mask") (roundrect_rratio 0.1886792453)
       (net 1 "Net-(C1-Pad1)") (pintype "passive"))
-    (pad "2" smd roundrect (at 1.5375 0) (size 1.325 2.35) (layers "F.Cu" "F.Paste" "F.Mask") (roundrect_rratio 0.188679)
+    (pad "2" smd roundrect (at 1.5375 0) (size 1.325 2.35) (layers "F.Cu" "F.Paste" "F.Mask") (roundrect_rratio 0.1886792453)
       (net 2 "Net-(J3-Pin_1)") (pintype "passive"))
     (model "${KICAD6_3DMODEL_DIR}/Capacitor_Tantalum_SMD.3dshapes/CP_EIA-3528-12_Kemet-T.wrl"
@@
     (fp_line (start 1.75 1.4) (end 1.75 -1.4)
       (stroke (width 0.1) (type solid)) (layer "F.Fab"))
-    (pad "1" smd roundrect (at -1.5375 0) (size 1.325 2.35) (layers "F.Cu" "F.Paste" "F.Mask") (roundrect_rratio 0.188679)
+    (pad "1" smd roundrect (at -1.5375 0) (size 1.325 2.35) (layers "F.Cu" "F.Paste" "F.Mask") (roundrect_rratio 0.1886792453)
       (net 3 "Net-(C2-Pad1)") (pintype "passive"))
-    (pad "2" smd roundrect (at 1.5375 0) (size 1.325 2.35) (layers "F.Cu" "F.Paste" "F.Mask") (roundrect_rratio 0.188679)
+    (pad "2" smd roundrect (at 1.5375 0) (size 1.325 2.35) (layers "F.Cu" "F.Paste" "F.Mask") (roundrect_rratio 0.1886792453)
       (net 4 "Net-(J4-Pin_1)") (pintype "passive"))
     (model "${KICAD6_3DMODEL_DIR}/Capacitor_Tantalum_SMD.3dshapes/CP_EIA-3528-12_Kemet-T.wrl"
@@
     (fp_line (start 1 0.625) (end -1 0.625)
       (stroke (width 0.1) (type solid)) (layer "F.Fab"))
-    (pad "1" smd roundrect (at -0.9125 0) (size 1.025 1.4) (layers "F.Cu" "F.Paste" "F.Mask") (roundrect_rratio 0.243902)
+    (pad "1" smd roundrect (at -0.9125 0) (size 1.025 1.4) (layers "F.Cu" "F.Paste" "F.Mask") (roundrect_rratio 0.243902439)
       (net 5 "Net-(J1-Pin_1)") (pintype "passive"))
-    (pad "2" smd roundrect (at 0.9125 0) (size 1.025 1.4) (layers "F.Cu" "F.Paste" "F.Mask") (roundrect_rratio 0.243902)
+    (pad "2" smd roundrect (at 0.9125 0) (size 1.025 1.4) (layers "F.Cu" "F.Paste" "F.Mask") (roundrect_rratio 0.243902439)
       (net 1 "Net-(C1-Pad1)") (pintype "passive"))
     (model "${KICAD6_3DMODEL_DIR}/Resistor_SMD.3dshapes/R_0805_2012Metric.wrl"
@@
   (gr_rect (start 105.6386 72.7456) (end 115.062 80.2132)
     (stroke (width 0.1) (type default)) (fill none) (layer "Edge.Cuts"))
-  (gr_text "JLCJLCJLCJLC" (at 114.5794 78.3336) (layer "B.SilkS")
-    (effects (font (size 0.8 0.8) (thickness 0.15)) (justify left bottom mirror))
-  )
-  (gr_text "SG/MD \nModel 2 & 3 \nS-Video\nBy joshman196" (at 115.0112 76.8604) (layer "B.SilkS")
+  (gr_text "JLCJLCJLCJLC" (at 115 80.1) (layer "B.SilkS")
+    (effects (font (size 0.7 0.7) (thickness 0.125) bold) (justify left bottom mirror))
+  )
+  (gr_text "SG/MD \nModel 2 & 3 \nS-Video\nBy joshman196" (at 115.0112 77.85) (layer "B.SilkS")
     (effects (font (size 0.65 0.65) (thickness 0.1)) (justify left bottom mirror))
   )
@@
     (effects (font (size 0.5 0.5) (thickness 0.125) bold) (justify left bottom))
   )
-  (gr_text "GND" (at 111.7092 76.7588) (layer "F.SilkS")
+  (gr_text "YCGND" (at 110.95 76.75) (layer "F.SilkS")
     (effects (font (size 0.4 0.4) (thickness 0.1) bold) (justify left bottom))
   )
@@
   (segment (start 106.68 79.6798) (end 106.68 78.4352) (width 0.65) (layer "F.Cu") (net 6))
   (segment (start 114.01 76.49) (end 114.02 76.5) (width 0.65) (layer "F.Cu") (net 7))
-  (segment (start 106.68 76.49) (end 114.01 76.49) (width 0.65) (layer "F.Cu") (net 7))
-  (via (at 111.4044 79.248) (size 0.8) (drill 0.4) (layers "F.Cu" "B.Cu") (free) (net 7))
+  (via (at 110.4 76.5) (size 0.8) (drill 0.4) (layers "F.Cu" "B.Cu") (free) (net 7))
   (zone (net 7) (net_name "GND") (layer "F.Cu") (hatch edge 0.5)
-    (connect_pads (clearance 0.1))
+    (connect_pads yes (clearance 0.1))
     (min_thickness 0.25) (filled_areas_thickness no)
     (fill yes (thermal_gap 0.5) (thermal_bridge_width 0.5))
